File: PeltierSwitchingMainBoard_control.sch (KiCad schematic (older format))
At the start: 24 parts, among them J3 Molex Micro Lock (1.25mm 1.5A), J4 Conn_01x14, U1 HIP4080A

Commit message: Removed custom footprint
Signed-off-by: bebenlebricolo <benoittarrade@hotmail.fr>
Parts:
- J4: footprint PeltierSwitchingMainBoard_control:Mezzanine_board_14contacts -> Connector_PinHeader_2.54mm:PinHeader_1x14_P2.54mm_Vertical
Changed lines of the file:
@@
 F 0 "J4" H 6780 2492 50  0000 L CNN
 F 1 "Conn_01x14" H 6780 2401 50  0000 L CNN
-F 2 "PeltierSwitchingMainBoard_control:Mezzanine_board_14contacts" H 6700 2500 50  0001 C CNN
+F 2 "Connector_PinHeader_2.54mm:PinHeader_1x14_P2.54mm_Vertical" H 6700 2500 50  0001 C CNN
 F 3 "~" H 6700 2500 50  0001 C CNN
 	1    6700 2500

Commit message: Updated silkscreen and exported Gerber files
Signed-off-by: bebenlebricolo <benoittarrade@hotmail.fr>
Other:
- note added: "1.0"
- note added: "10/09/2021 (dd/mm/yyyy)"
- note added: "Beer thermoregulation system (main board, control section)"
- note added: "Designed by Benoit Tarrade\n(alias bebenlebricolo)\nhttps://github.com/bebenlebricolo"
- note added: "This board is a mezzanine board for the beer thermoregulation system\n main board. It was designed to workaround the single-sided Aluminum limitations\nof the power board and use a regular double sided FR4 board.\nThis board handles signal processing and mosfet driving using the hip4080a IC.\nInput signal comes from another logic board from which a PWM signal \nis generated (either by a µC or a N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"
Changed lines of the file:
@@
 Text Label 6500 2900 2    50   ~ 0
 Vcc
+Text Notes 7350 7500 0    79   Italic 0
+Beer thermoregulation system (main board, control section)
+Text Notes 10575 7625 0    50   Italic 0
+1.0
+Text Notes 8175 7625 0    50   Italic 0
+10/09/2021 (dd/mm/yyyy)
+Text Notes 7000 7075 0    50   ~ 0
+This board is a mezzanine board for the beer thermoregulation system\n main board. It was designed to workaround the single-sided Aluminum limitations\nof the power board and use a regular double sided FR4 board.\nThis board handles signal processing and mosfet driving using the hip4080a IC.\nInput signal comes from another logic board from which a PWM signal \nis generated (either by a µC or a NE555 timer).
+Text Notes 9775 6450 0    50   Italic 0
+Designed by Benoit Tarrade\n(alias bebenlebricolo)\nhttps://github.com/bebenlebricolo
 $EndSCHEMATC
